Commit message: Fixed joint names and imported meshes so it works in gazebo

File: Simulation/PAROL6.urdf (robot description, URDF)
Before this commit: robot PAROL6, 7 links, 6 joints
Links:
- removed link L1
- removed link L2
- removed link L3
- removed link L4
- removed link L5
- removed link L6
- added link link_L1, mass 0.644800830530233; collision mesh filename=package://PAROL6/meshes/L1.STL; visual mesh filename=package://PAROL6/meshes/L1.STL
- added link link_L2, mass 0.512334779399788; collision mesh filename=package://PAROL6/meshes/L2.STL; visual mesh filename=package://PAROL6/meshes/L2.STL
- added link link_L3, mass 0.550970997806044; collision mesh filename=package://PAROL6/meshes/L3.STL; visual mesh filename=package://PAROL6/meshes/L3.STL
- added link link_L4, mass 0.39346362633915; collision mesh filename=package://PAROL6/meshes/L4.STL; visual mesh filename=package://PAROL6/meshes/L4.STL
- added link link_L5, mass 0.185171777001718; collision mesh filename=package://PAROL6/meshes/L5.STL; visual mesh filename=package://PAROL6/meshes/L5.STL
- added link link_L6, mass 0.0703261410665101; collision mesh filename=package://PAROL6/meshes/L6.STL; visual mesh filename=package://PAROL6/meshes/L6.STL
Joints:
- removed joint L1
- removed joint L2
- removed joint L3
- removed joint L4
- removed joint L5
- removed joint L6
- added joint joint_L1: type revolute, parent base_link, child link_L1, origin xyz=0 0 0 rpy=0 0 0, axis 0 0 1, limit lower=0 upper=0 effort=0 velocity=0
- added joint joint_L2: type revolute, parent link_L1, child link_L2, origin xyz=0.0234207210610375 0 0.1105 rpy=-1.5707963267949 0 0, axis 0 0 1, limit lower=0 upper=0 effort=0 velocity=0
- added joint joint_L3: type revolute, parent link_L2, child link_L3, origin xyz=0 -0.18 0 rpy=3.1416 0 -1.5708, axis 0 0 -1, limit lower=0 upper=0 effort=0 velocity=0
- added joint joint_L4: type revolute, parent link_L3, child link_L4, origin xyz=0.0435 0 0 rpy=1.5707963267949 0 3.14159265358979, axis 0 0 -1, limit lower=0 upper=0 effort=0 velocity=0
- added joint joint_L5: type revolute, parent link_L4, child link_L5, origin xyz=0 0 -0.17635 rpy=-1.5708 0 0, axis 0 0 -1, limit lower=0 upper=0 effort=0 velocity=0
- added joint joint_L6: type continuous, parent link_L5, child link_L6, origin xyz=0 0 0 rpy=1.5708 0 0, axis 0 0 -1, limit lower=0 upper=0 effort=0 velocity=0
