Commit message: pyBullet working to rotate bot

File: Simulation/robot.urdf (robot description, URDF)
Before this commit: robot PAROL6, 7 links, 6 joints
Joints:
- joint joint_L1: limit lower=0 upper=0 effort=0 velocity=0 -> lower=0 upper=2 effort=15 velocity=0.5
- joint joint_L2: limit lower=0 upper=0 effort=0 velocity=0 -> lower=0 upper=2 effort=15 velocity=0.5
- joint joint_L3: limit lower=0 upper=0 effort=0 velocity=0 -> lower=0 upper=2 effort=15 velocity=0.5
- joint joint_L4: limit lower=0 upper=0 effort=0 velocity=0 -> lower=0 upper=2 effort=15 velocity=0.5
- joint joint_L5: limit lower=0 upper=0 effort=0 velocity=0 -> lower=0 upper=2 effort=15 velocity=0.5
- joint joint_L6: limit lower=0 upper=0 effort=0 velocity=0 -> lower=0 upper=2 effort=15 velocity=0.5

Commit message: I got the bot to move but not like that. And when it moves slightly, the whole bot tips over. So I decided to lock the base onto the floor, but now the bot won't move at all. I've been unable to make the bot move again. Also had to change one of the joints from 'continuous' to 'revolute' so that an ikpy function would work. On that note, I'm using ikpy to get the positions, then just moving it using pybullet.

File: Simulation/robot.urdf (robot description, URDF)
Before this commit: robot PAROL6, 7 links, 6 joints
Joints:
- joint joint_L6: type continuous -> revolute

Commit message: Controller works with simulation

File: Simulation/robot.urdf (robot description, URDF)
Before this commit: robot PAROL6, 7 links, 6 joints
Joints:
- joint joint_L1: limit lower=0 upper=2 effort=15 velocity=0.5 -> lower=-2 upper=2 effort=15 velocity=0.5
- joint joint_L2: limit lower=0 upper=2 effort=15 velocity=0.5 -> lower=-2 upper=2 effort=15 velocity=0.5
- joint joint_L3: limit lower=0 upper=2 effort=15 velocity=0.5 -> lower=-2 upper=2 effort=15 velocity=0.5
- joint joint_L4: limit lower=0 upper=2 effort=15 velocity=0.5 -> lower=-2 upper=2 effort=15 velocity=0.5
- joint joint_L5: limit lower=0 upper=2 effort=15 velocity=0.5 -> lower=-2 upper=2 effort=15 velocity=0.5
- joint joint_L6: limit lower=0 upper=2 effort=15 velocity=0.5 -> lower=-2 upper=2 effort=15 velocity=0.5

Commit message: Added new claw to simulation and fixed requirements.txt

File: Simulation/robot.urdf (robot description, URDF)
Before this commit: robot PAROL6, 7 links, 6 joints
Links:
- link link_L6: geometry collision mesh filename=package://PAROL6/meshes/claw.stl scale=0.001 0.001 0.001; visual mesh filename=package://PAROL6/meshes/claw.stl scale=0.001 0.001 0.001
Joints:
- joint joint_L6: axis 0 0 -1 -> 0 1 0; origin xyz=0 0 0 rpy=1.5708 0 0 -> xyz=0 0.1 0 rpy=0 1.5708 0
